Commit message: ADD world link,, table joint, REMOVED multi arm param

File: urdf/bimanual.urdf.xacro (robot description, xacro)
@@ -2,4 +2,10 @@
 <robot xmlns:xacro="http://www.ros.org/wiki/xacro" name="idra_bimanual_setup">
   <xacro:include filename="$(find franka_description)/robots/common/franka_robot.xacro"/>
+  <link name="world"/>
+  <joint name="world_joint" type="fixed">
+    <origin rpy="0 0 0" xyz="0 0 0.2"/>
+    <parent link="world"/>
+    <child link="table"/>
+  </joint>
   <!--  _____     _     _       -->
   <!-- |_   _|_ _| |__ | | ___  -->
@@ -22,4 +28,10 @@
       <material name="tablematerial"/>
     </visual>
+    <collision>
+      <geometry>
+        <box size="1.2 0.8 0.2"/>
+      </geometry>
+      <origin xyz="0.6 0.4 -0.1"/>
+    </collision>
   </link>
   <link name="robot1_plate">
@@ -91,11 +103,11 @@
                       ros2_control="$(arg ros2_control)"
                       robot_ip="192.160.100.11"
-                      arm_prefix="franka1"
+                      arm_prefix="franka1_"
                       connected_to="franka1_base"
-                      multi_arm="true"
                       no_prefix="false"
                       use_fake_hardware="$(arg use_fake_hardware)"
                       fake_sensor_commands="$(arg fake_sensor_commands)"
-                      gazebo_effort="$(arg gazebo_effort)">
+                      gazebo_effort="$(arg gazebo_effort)"
+                      >
   </xacro:franka_robot>
   <!-- Dimensions taken from technical drawing of Franka plate and custom designed plate, do not touch -->
@@ -122,11 +134,11 @@
                       ros2_control="$(arg ros2_control)"
                       robot_ip="192.160.100.12"
-                      arm_prefix="franka2"
+                      arm_prefix="franka2_"
                       connected_to="franka2_base"
-                      multi_arm="true"
                       no_prefix="false"
                       use_fake_hardware="$(arg use_fake_hardware)"
                       fake_sensor_commands="$(arg fake_sensor_commands)"
-                      gazebo_effort="$(arg gazebo_effort)">
+                      gazebo_effort="$(arg gazebo_effort)"
+                      >
   </xacro:franka_robot>
   <!-- Dimensions taken from technical drawing of Franka plate and custom designed plate, do not touch -->

Commit message: ADD Custom ros2_control

File: urdf/bimanual.urdf.xacro (robot description, xacro)
@@ -86,6 +86,6 @@
   <xacro:arg name="gazebo_effort" default="false" />
   <xacro:arg name="multi_arm" default="true" />
-  <xacro:arg name="franka1_ip" default="192.168.100.11" />
-  <xacro:arg name="franka2_ip" default="192.168.100.12" />
+  <xacro:arg name="franka1_ip" default="192.160.100.11" />
+  <xacro:arg name="franka2_ip" default="192.160.100.12" />
   <xacro:arg name="controller_path" default="$(find idra_franka_launch)/config/basic_controllers.yaml" />
   <!--  _____                _         _  -->
@@ -151,4 +151,63 @@
     <origin xyz="0.145 0.107 0.018" rpy="0 0 ${-pi/2}"/>
   </joint>
+  <!-- TODO: add if based on ros2_control arg -->
+  <ros2_control name="FrankaBimanualHardwareInterface" type="system">
+    <hardware>
+      <xacro:if value="$(arg use_fake_hardware)">
+        <plugin>fake_components/GenericSystem</plugin>
+        <param name="mock_sensor_commands">$(arg use_fake_hardware)</param>
+        <param name="state_following_offset">0.0</param>
+      </xacro:if>
+      <xacro:if value="$(arg gazebo)">
+        <plugin>franka_ign_ros2_control/IgnitionSystem</plugin>
+      </xacro:if>
+      <xacro:if value="$(eval not use_fake_hardware and not gazebo)">
+        <plugin>franka_bimanual_hardware_interface/FrankaBimanualHardwareInterface</plugin>
+        <param name="franka1_ip">$(arg franka1_ip)</param>
+        <param name="franka2_ip">$(arg franka2_ip)</param>
+      </xacro:if>
+    </hardware>
+    <!-- Joint position, velocity and effort interfaces -->
+    <xacro:macro name="configure_joint" params="joint_name initial_position">
+      <joint name="${joint_name}">
+        <!--
+          deactivated for gazebo velocity and position interface due to a bug
+          https://github.com/ros-controls/gz_ros2_control/issues/343
+          Command Interfaces -->
+          <command_interface name="position"/>
+          <command_interface name="velocity"/>
+        <xacro:if value="$(eval not gazebo or gazebo_effort)">
+          <command_interface name="effort"/>
+        </xacro:if>
+        <!-- State Interfaces -->
+        <state_interface name="position">
+          <param name="initial_value">${initial_position}</param>
+        </state_interface>
+        <state_interface name="velocity"/>
+          <param name="initial_value">0.0</param>
+        <state_interface name="effort"/>
+      </joint>
+    </xacro:macro>
+    <xacro:configure_joint joint_name="franka1_fr3_joint1" initial_position="0.0"/>
+    <xacro:configure_joint joint_name="franka1_fr3_joint2" initial_position="${-pi/4}"/>
+    <xacro:configure_joint joint_name="franka1_fr3_joint3" initial_position="0.0"/>
+    <xacro:configure_joint joint_name="franka1_fr3_joint4" initial_position="${-3*pi/4}"/>
+    <xacro:configure_joint joint_name="franka1_fr3_joint5" initial_position="0.0"/>
+    <xacro:configure_joint joint_name="franka1_fr3_joint6" initial_position="${pi/2}"/>
+    <xacro:configure_joint joint_name="franka1_fr3_joint7" initial_position="${pi/4}"/>
+    <xacro:if value="$(eval gazebo and hand)">
+      <xacro:configure_joint joint_name="$franka1_fr3_finger_joint1" initial_position="0.0" />
+    </xacro:if>
+    <xacro:configure_joint joint_name="franka2_fr3_joint1" initial_position="0.0"/>
+    <xacro:configure_joint joint_name="franka2_fr3_joint2" initial_position="${-pi/4}"/>
+    <xacro:configure_joint joint_name="franka2_fr3_joint3" initial_position="0.0"/>
+    <xacro:configure_joint joint_name="franka2_fr3_joint4" initial_position="${-3*pi/4}"/>
+    <xacro:configure_joint joint_name="franka2_fr3_joint5" initial_position="0.0"/>
+    <xacro:configure_joint joint_name="franka2_fr3_joint6" initial_position="${pi/2}"/>
+    <xacro:configure_joint joint_name="franka2_fr3_joint7" initial_position="${pi/4}"/>
+    <xacro:if value="$(eval gazebo and hand)">
+      <xacro:configure_joint joint_name="$franka2_fr3_finger_joint1" initial_position="0.0" />
+    </xacro:if>
+  </ros2_control>
   <xacro:if value="$(arg gazebo)">
   <gazebo>
