Commit message: ADD Cartesian velocity interfaces

File: idra_franka_launch/urdf/bimanual.urdf.xacro (robot description, xacro)
@@ -192,4 +192,10 @@
       </joint>
     </xacro:macro>
+    <xacro:macro name="general_purpose_io" params="prefix command_interface index">
+      <gpio name="${prefix}">
+        <command_interface name="${command_interface}"/>
+        <!-- <param name="index">${index}</param> -->
+      </gpio>
+    </xacro:macro>
     <xacro:configure_joint joint_name="franka1_fr3_joint1" initial_position="0.0"/>
     <xacro:configure_joint joint_name="franka1_fr3_joint2" initial_position="${-pi/4}"/>
@@ -200,5 +206,5 @@
     <xacro:configure_joint joint_name="franka1_fr3_joint7" initial_position="${pi/4}"/>
     <xacro:if value="$(eval gazebo and hand)">
-      <xacro:configure_joint joint_name="$franka1_fr3_finger_joint1" initial_position="0.0" />
+      <xacro:configure_joint joint_name="franka1_fr3_finger_joint1" initial_position="0.0" />
     </xacro:if>
     <xacro:configure_joint joint_name="franka2_fr3_joint1" initial_position="0.0"/>
@@ -210,6 +216,19 @@
     <xacro:configure_joint joint_name="franka2_fr3_joint7" initial_position="${pi/4}"/>
     <xacro:if value="$(eval gazebo and hand)">
-      <xacro:configure_joint joint_name="$franka2_fr3_finger_joint1" initial_position="0.0" />
+      <xacro:configure_joint joint_name="franka2_fr3_finger_joint1" initial_position="0.0" />
     </xacro:if>
+    <!-- Cartesian velocity interfaces -->
+    <xacro:general_purpose_io prefix="franka1_vx" command_interface="cartesian_velocity" index="0"/>
+    <xacro:general_purpose_io prefix="franka1_vy" command_interface="cartesian_velocity" index="1"/>
+    <xacro:general_purpose_io prefix="franka1_vz" command_interface="cartesian_velocity" index="2"/>
+    <xacro:general_purpose_io prefix="franka1_wx" command_interface="cartesian_velocity" index="3"/>
+    <xacro:general_purpose_io prefix="franka1_wy" command_interface="cartesian_velocity" index="4"/>
+    <xacro:general_purpose_io prefix="franka1_wz" command_interface="cartesian_velocity" index="5"/>
+    <xacro:general_purpose_io prefix="franka2_vx" command_interface="cartesian_velocity" index="0"/>
+    <xacro:general_purpose_io prefix="franka2_vy" command_interface="cartesian_velocity" index="1"/>
+    <xacro:general_purpose_io prefix="franka2_vz" command_interface="cartesian_velocity" index="2"/>
+    <xacro:general_purpose_io prefix="franka2_wx" command_interface="cartesian_velocity" index="3"/>
+    <xacro:general_purpose_io prefix="franka2_wy" command_interface="cartesian_velocity" index="4"/>
+    <xacro:general_purpose_io prefix="franka2_wz" command_interface="cartesian_velocity" index="5"/>
   </ros2_control>
   <xacro:if value="$(arg gazebo)">

Commit message: ADD Cartesian pose interface

File: idra_franka_launch/urdf/bimanual.urdf.xacro (robot description, xacro)
@@ -223,4 +223,19 @@
     <xacro:general_purpose_io prefix="franka2_joint_3_position" command_interface="elbow_command" index="0"/>
     <xacro:general_purpose_io prefix="franka2_joint_4_sign" command_interface="elbow_command" index="1"/>
+    <!-- Cartesian position interfaces -->
+    <xacro:macro name="loop" params="i">
+      <xacro:unless value="${i == 16}">
+        <xacro:general_purpose_io prefix="franka1_${i}" command_interface="cartesian_pose_command" index="${i}"/>
+        <xacro:loop i="${i+1}"/>
+      </xacro:unless>
+    </xacro:macro>
+    <xacro:loop i="0"/>
+    <xacro:macro name="loop" params="i">
+      <xacro:unless value="${i == 16}">
+        <xacro:general_purpose_io prefix="franka2_${i}" command_interface="cartesian_pose_command" index="${i}"/>
+        <xacro:loop i="${i+1}"/>
+      </xacro:unless>
+    </xacro:macro>
+    <xacro:loop i="0"/>
     <!-- Cartesian velocity interfaces -->
     <xacro:general_purpose_io prefix="franka1_vx" command_interface="cartesian_velocity" index="0"/>

Commit message: ADD Macro interface_spawner for the urdf

File: idra_franka_launch/urdf/bimanual.urdf.xacro (robot description, xacro)
@@ -154,21 +154,5 @@
   </joint>
   <!-- TODO: add if based on ros2_control arg -->
-  <ros2_control name="FrankaBimanualHardwareInterface" type="system">
-    <hardware>
-      <xacro:if value="$(arg use_fake_hardware)">
-        <plugin>fake_components/GenericSystem</plugin>
-        <param name="mock_sensor_commands">$(arg use_fake_hardware)</param>
-        <param name="state_following_offset">0.0</param>
-      </xacro:if>
-      <xacro:if value="$(arg gazebo)">
-        <plugin>franka_ign_ros2_control/IgnitionSystem</plugin>
-      </xacro:if>
-      <xacro:if value="$(eval not use_fake_hardware and not gazebo)">
-        <plugin>franka_bimanual_hardware_interface/FrankaBimanualHardwareInterface</plugin>
-        <param name="robot_names">franka1,franka2</param>
-        <param name="robot_ips">$(arg franka1_ip),$(arg franka2_ip)</param>
-        <param name="limit_override">$(arg limit_override)</param>
-      </xacro:if>
-    </hardware>
+  <xacro:macro name="interface_spawner" params="robot_name">
     <!-- Joint position, velocity and effort interfaces -->
     <xacro:macro name="configure_joint" params="joint_name initial_position">
@@ -198,40 +182,21 @@
       </gpio>
     </xacro:macro>
-    <xacro:configure_joint joint_name="franka1_fr3_joint1" initial_position="0.0"/>
-    <xacro:configure_joint joint_name="franka1_fr3_joint2" initial_position="${-pi/4}"/>
-    <xacro:configure_joint joint_name="franka1_fr3_joint3" initial_position="0.0"/>
-    <xacro:configure_joint joint_name="franka1_fr3_joint4" initial_position="${-3*pi/4}"/>
-    <xacro:configure_joint joint_name="franka1_fr3_joint5" initial_position="0.0"/>
-    <xacro:configure_joint joint_name="franka1_fr3_joint6" initial_position="${pi/2}"/>
-    <xacro:configure_joint joint_name="franka1_fr3_joint7" initial_position="${pi/4}"/>
+    <xacro:configure_joint joint_name="${robot_name}_fr3_joint1" initial_position="0.0"/>
+    <xacro:configure_joint joint_name="${robot_name}_fr3_joint2" initial_position="${-pi/4}"/>
+    <xacro:configure_joint joint_name="${robot_name}_fr3_joint3" initial_position="0.0"/>
+    <xacro:configure_joint joint_name="${robot_name}_fr3_joint4" initial_position="${-3*pi/4}"/>
+    <xacro:configure_joint joint_name="${robot_name}_fr3_joint5" initial_position="0.0"/>
+    <xacro:configure_joint joint_name="${robot_name}_fr3_joint6" initial_position="${pi/2}"/>
+    <xacro:configure_joint joint_name="${robot_name}_fr3_joint7" initial_position="${pi/4}"/>
     <xacro:if value="$(eval gazebo and hand)">
-      <xacro:configure_joint joint_name="franka1_fr3_finger_joint1" initial_position="0.0" />
-    </xacro:if>
-    <xacro:configure_joint joint_name="franka2_fr3_joint1" initial_position="0.0"/>
-    <xacro:configure_joint joint_name="franka2_fr3_joint2" initial_position="${-pi/4}"/>
-    <xacro:configure_joint joint_name="franka2_fr3_joint3" initial_position="0.0"/>
-    <xacro:configure_joint joint_name="franka2_fr3_joint4" initial_position="${-3*pi/4}"/>
-    <xacro:configure_joint joint_name="franka2_fr3_joint5" initial_position="0.0"/>
-    <xacro:configure_joint joint_name="franka2_fr3_joint6" initial_position="${pi/2}"/>
-    <xacro:configure_joint joint_name="franka2_fr3_joint7" initial_position="${pi/4}"/>
-    <xacro:if value="$(eval gazebo and hand)">
-      <xacro:configure_joint joint_name="franka2_fr3_finger_joint1" initial_position="0.0" />
+      <xacro:configure_joint joint_name="${robot_name}_fr3_finger_joint1" initial_position="0.0" />
     </xacro:if>
     <!-- Elbow interfaces -->
-    <xacro:general_purpose_io prefix="franka1_joint_3_position" command_interface="elbow_command" index="0"/>
-    <xacro:general_purpose_io prefix="franka1_joint_4_sign" command_interface="elbow_command" index="1"/>
-    <xacro:general_purpose_io prefix="franka2_joint_3_position" command_interface="elbow_command" index="0"/>
-    <xacro:general_purpose_io prefix="franka2_joint_4_sign" command_interface="elbow_command" index="1"/>
+    <xacro:general_purpose_io prefix="${robot_name}_joint_3_position" command_interface="elbow_command" index="0"/>
+    <xacro:general_purpose_io prefix="${robot_name}_joint_4_sign" command_interface="elbow_command" index="1"/>
     <!-- Cartesian position interfaces -->
     <xacro:macro name="loop" params="i">
       <xacro:unless value="${i == 16}">
-        <xacro:general_purpose_io prefix="franka1_${i}" command_interface="cartesian_pose_command" index="${i}"/>
-        <xacro:loop i="${i+1}"/>
-      </xacro:unless>
-    </xacro:macro>
-    <xacro:loop i="0"/>
-    <xacro:macro name="loop" params="i">
-      <xacro:unless value="${i == 16}">
-        <xacro:general_purpose_io prefix="franka2_${i}" command_interface="cartesian_pose_command" index="${i}"/>
+        <xacro:general_purpose_io prefix="${robot_name}_${i}" command_interface="cartesian_pose_command" index="${i}"/>
         <xacro:loop i="${i+1}"/>
       </xacro:unless>
@@ -239,16 +204,30 @@
     <xacro:loop i="0"/>
     <!-- Cartesian velocity interfaces -->
-    <xacro:general_purpose_io prefix="franka1_vx" command_interface="cartesian_velocity" index="0"/>
-    <xacro:general_purpose_io prefix="franka1_vy" command_interface="cartesian_velocity" index="1"/>
-    <xacro:general_purpose_io prefix="franka1_vz" command_interface="cartesian_velocity" index="2"/>
-    <xacro:general_purpose_io prefix="franka1_wx" command_interface="cartesian_velocity" index="3"/>
-    <xacro:general_purpose_io prefix="franka1_wy" command_interface="cartesian_velocity" index="4"/>
-    <xacro:general_purpose_io prefix="franka1_wz" command_interface="cartesian_velocity" index="5"/>
-    <xacro:general_purpose_io prefix="franka2_vx" command_interface="cartesian_velocity" index="0"/>
-    <xacro:general_purpose_io prefix="franka2_vy" command_interface="cartesian_velocity" index="1"/>
-    <xacro:general_purpose_io prefix="franka2_vz" command_interface="cartesian_velocity" index="2"/>
-    <xacro:general_purpose_io prefix="franka2_wx" command_interface="cartesian_velocity" index="3"/>
-    <xacro:general_purpose_io prefix="franka2_wy" command_interface="cartesian_velocity" index="4"/>
-    <xacro:general_purpose_io prefix="franka2_wz" command_interface="cartesian_velocity" index="5"/>
+    <xacro:general_purpose_io prefix="${robot_name}_vx" command_interface="cartesian_velocity" index="0"/>
+    <xacro:general_purpose_io prefix="${robot_name}_vy" command_interface="cartesian_velocity" index="1"/>
+    <xacro:general_purpose_io prefix="${robot_name}_vz" command_interface="cartesian_velocity" index="2"/>
+    <xacro:general_purpose_io prefix="${robot_name}_wx" command_interface="cartesian_velocity" index="3"/>
+    <xacro:general_purpose_io prefix="${robot_name}_wy" command_interface="cartesian_velocity" index="4"/>
+    <xacro:general_purpose_io prefix="${robot_name}_wz" command_interface="cartesian_velocity" index="5"/>
+  </xacro:macro>
+  <ros2_control name="FrankaBimanualHardwareInterface" type="system">
+    <hardware>
+      <xacro:if value="$(arg use_fake_hardware)">
+        <plugin>fake_components/GenericSystem</plugin>
+        <param name="mock_sensor_commands">$(arg use_fake_hardware)</param>
+        <param name="state_following_offset">0.0</param>
+      </xacro:if>
+      <xacro:if value="$(arg gazebo)">
+        <plugin>franka_ign_ros2_control/IgnitionSystem</plugin>
+      </xacro:if>
+      <xacro:if value="$(eval not use_fake_hardware and not gazebo)">
+        <plugin>franka_bimanual_hardware_interface/FrankaBimanualHardwareInterface</plugin>
+        <param name="robot_names">franka1,franka2</param>
+        <param name="robot_ips">$(arg franka1_ip),$(arg franka2_ip)</param>
+        <param name="limit_override">$(arg limit_override)</param>
+      </xacro:if>
+    </hardware>
+    <xacro:interface_spawner robot_name="franka1"/>
+    <xacro:interface_spawner robot_name="franka2"/>
   </ros2_control>
   <xacro:if value="$(arg gazebo)">

Commit message: UPDATE urdf, maganed to remove franka_base and aut_spawned word frames

File: idra_franka_launch/urdf/bimanual.urdf.xacro (robot description, xacro)
@@ -109,5 +109,6 @@
                       robot_ip="$(arg franka1_ip)"
                       arm_prefix="franka1_"
-                      connected_to="franka1_base"
+                      parent=""
+                      connected_to=""
                       no_prefix="false"
                       use_fake_hardware="$(arg use_fake_hardware)"
@@ -120,5 +121,5 @@
   <joint name="plate_to_franka1" type="fixed">
     <parent link="robot1_plate"/>
-    <child link="franka1_base"/>
+    <child link="franka1_fr3_link0"/>
     <origin xyz="0.145 0.107 0.018" rpy="0 0 ${-pi/2}"/>
   </joint>
@@ -141,5 +142,6 @@
                       robot_ip="$(arg franka2_ip)"
                       arm_prefix="franka2_"
-                      connected_to="franka2_base"
+                      parent=""
+                      connected_to=""
                       no_prefix="false"
                       use_fake_hardware="$(arg use_fake_hardware)"
@@ -152,5 +154,5 @@
   <joint name="plate_to_franka2" type="fixed">
     <parent link="robot2_plate"/>
-    <child link="franka2_base"/>
+    <child link="franka2_fr3_link0"/>
     <origin xyz="0.145 0.107 0.018" rpy="0 0 ${-pi/2}"/>
   </joint>
